Commit message: improved grasp candidates

File: ACRLUnity/Assets/Prefabs/arf_urdf/ar4.urdf (robot description, URDF)
Before this commit: robot mk3, 12 links, 11 joints
Joints:
- joint gripper_jaw1_joint: limit lower=0 upper=0.014 effort=-1 velocity=1.0 -> lower=0 upper=0.014 effort=5000 velocity=1.0
- joint gripper_jaw2_joint: limit lower=0 upper=0.014 effort=1000 velocity=1.0 -> lower=0 upper=0.014 effort=5000 velocity=1.0
