Commit message: feat: Update Unity scene defaults, refine ROS MoveIt joint limits, improve dashboard object rendering, and enhance server shutdown for ROS Docker.

File: rosUnityIntegration/ar4_moveit_config/urdf/ar4.urdf (robot description, URDF)
Before this commit: robot mk3, 12 links, 11 joints
Joints:
- joint joint_4: limit lower=-3.141592653589793 upper=3.141592653589793 effort=-1 velocity=1.0472 -> lower=-3.1405926535897932 upper=3.1405926535897932 effort=-1 velocity=1.0472
- joint joint_6: limit lower=-3.141592653589793 upper=3.141592653589793 effort=-1 velocity=1.0472 -> lower=-3.1405926535897932 upper=3.1405926535897932 effort=-1 velocity=1.0472
